File: src/main/resources/kicad/DigiSim/6bitincdec.kicad_sch (KiCad schematic)
At the start: 7 parts

Commit message: Hierarchical Scheme added
Connections:
- net Decrement: now reaches or4.B, or5.B, or6.B, or7.B, or8.B, or9.B
- net incdec4/Dec0-in: now reaches and3.F, or8.O
- net incdec4/Dec1-in: now reaches and3.G, or9.O
- net D5: now reaches or9.A
- net D4: now reaches or8.A
- net incdec2/D0-in renamed D0
- net incdec2/D1-in renamed D1
- net incdec3/D0-in renamed D2
- net incdec3/D1-in renamed D3
Other:
- added sheet incdec4 (incdec2.kicad_sch)
- moved on the sheet: or9
