File: src/main/resources/kicad/DigiSim/incdec2.kicad_sch (KiCad schematic)
At the start: 4 parts

Commit message: Hierarchical Scheme added
Parts:
- renumbered and4 to and8, and5 to and9, or11 to or14, or10 to or15
Changed lines of the file:
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@@
 		(in_pos_files yes)
 		(dnp no)
-		(property "Reference" "or11"
+		(property "Reference" "or14"
 			(at 144.78 31.75 0)
 			(show_name no)
@@
 				(path "/da9e1665-5c64-4bd6-93fc-709c1dd71100/444aed17-0ebd-4591-b570-dca3e2ecef10"
 					(reference "or11")
+					(unit 1)
+				)
+				(path "/da9e1665-5c64-4bd6-93fc-709c1dd71100/c481537d-2184-4ee1-8037-13df63c28a4b"
+					(reference "or14")
 					(unit 1)
 				)
@@
 		(in_pos_files yes)
 		(dnp no)
-		(property "Reference" "and4"
+		(property "Reference" "and8"
 			(at 116.84 33.528 0)
 			(show_name no)
@@
 				(path "/da9e1665-5c64-4bd6-93fc-709c1dd71100/444aed17-0ebd-4591-b570-dca3e2ecef10"
 					(reference "and4")
+					(unit 1)
+				)
+				(path "/da9e1665-5c64-4bd6-93fc-709c1dd71100/c481537d-2184-4ee1-8037-13df63c28a4b"
+					(reference "and8")
 					(unit 1)
 				)
@@
 		(in_pos_files yes)
 		(dnp no)
-		(property "Reference" "or10"
+		(property "Reference" "or15"
 			(at 144.78 58.674 0)
 			(show_name no)
@@
 				(path "/da9e1665-5c64-4bd6-93fc-709c1dd71100/444aed17-0ebd-4591-b570-dca3e2ecef10"
 					(reference "or10")
+					(unit 1)
+				)
+				(path "/da9e1665-5c64-4bd6-93fc-709c1dd71100/c481537d-2184-4ee1-8037-13df63c28a4b"
+					(reference "or15")
 					(unit 1)
 				)
@@
 		(in_pos_files yes)
 		(dnp no)
-		(property "Reference" "and5"
+		(property "Reference" "and9"
 			(at 144.78 44.196 0)
 			(show_name no)
@@
 					(unit 1)
 				)
+				(path "/da9e1665-5c64-4bd6-93fc-709c1dd71100/c481537d-2184-4ee1-8037-13df63c28a4b"
+					(reference "and9")
+					(unit 1)
+				)
